Commit message: ok

File: src/inmoov_description/robots/inmoov_head_control.urdf.xacro (robot description, xacro)
@@ -79,36 +79,4 @@
     <child link="face_link"/>
   </joint>-->
-  <xacro:arm side="r" flip="1" covers="yes" />
-  <joint name="r_shoulder_out_joint" type="revolute">
-   <axis xyz="1 0 0"/>
-   <limit effort="1000.0" lower="${r_shoulder_out_joint_lower}" upper="${r_shoulder_out_joint_upper}" velocity="${r_shoulder_out_joint_velocity}" />
-   <origin rpy="0 0 0" xyz="0 -0.143 0.298"/>
-   <parent link="torso_link"/>
-   <child link="r_shoulder_base_link"/>
-  </joint>
-  <xacro:hand side="r" flip="1" covers="yes" />
-  <joint name="r_wrist_roll_joint" type="revolute">
-   <axis xyz="0 0 1"/>
-   <limit effort="1000.0" lower="${r_wrist_roll_joint_lower}" upper="${r_wrist_roll_joint_upper}" velocity="${r_wrist_roll_joint_velocity}" />
-   <origin rpy="0 0 0" xyz="-0.0144 0.01  -0.2885"/>
-   <parent link="r_forearm_link"/>
-   <child link="r_hand_link"/>
-  </joint>
-  <xacro:arm side="l" flip="-1" covers="yes" />
-  <joint name="l_shoulder_out_joint" type="revolute">
-   <axis xyz="1 0 0"/>
-   <limit effort="1000.0" lower="${l_shoulder_out_joint_lower}" upper="${l_shoulder_out_joint_upper}" velocity="${l_shoulder_out_joint_velocity}" />
-   <origin rpy="0 0 0" xyz="0 0.143 0.298"/>
-   <parent link="torso_link"/>
-   <child link="l_shoulder_base_link"/>
-  </joint>
-  <xacro:hand side="l" flip="-1" covers="yes" />
-  <joint name="l_wrist_roll_joint" type="revolute">
-   <axis xyz="0 0 1"/>
-   <limit effort="1000.0" lower="${l_wrist_roll_joint_lower}" upper="${l_wrist_roll_joint_upper}" velocity="${l_wrist_roll_joint_velocity}" />
-   <origin rpy="0 0 0" xyz="-0.0144 -0.01  -0.2885"/>
-   <parent link="l_forearm_link"/>
-   <child link="l_hand_link"/>
-  </joint>
   <xacro:robot_head name="RobotHead" prefix="" />
 </robot>

File: src/inmoov_description/robots/inmoov_right_hand.urdf.xacro (robot description, xacro)
@@ -19,8 +19,40 @@
   <joint name="base_to_hand_joint" type="revolute">
    <axis xyz="0 0 1"/>
-<limit effort="1000.0" lower="-3.14" upper="0" velocity="0.5"/>
-<origin rpy="0 0 0" xyz="0 0 0"/>
+    <limit effort="1000.0" lower="-3.14" upper="0" velocity="0.5"/>
+    <origin rpy="0 0 0" xyz="0 0 0"/>
     <parent link="base_link"/>
     <child link="r_hand_link"/>
   </joint>
+  <xacro:arm side="r" flip="1" covers="yes" />
+  <joint name="r_shoulder_out_joint" type="revolute">
+   <axis xyz="1 0 0"/>
+   <limit effort="1000.0" lower="${r_shoulder_out_joint_lower}" upper="${r_shoulder_out_joint_upper}" velocity="${r_shoulder_out_joint_velocity}" />
+   <origin rpy="0 0 0" xyz="0 -0.143 0.298"/>
+   <parent link="torso_link"/>
+   <child link="r_shoulder_base_link"/>
+  </joint>
+  <xacro:hand side="r" flip="1" covers="yes" />
+  <joint name="r_wrist_roll_joint" type="revolute">
+   <axis xyz="0 0 1"/>
+   <limit effort="1000.0" lower="${r_wrist_roll_joint_lower}" upper="${r_wrist_roll_joint_upper}" velocity="${r_wrist_roll_joint_velocity}" />
+   <origin rpy="0 0 0" xyz="-0.0144 0.01  -0.2885"/>
+   <parent link="r_forearm_link"/>
+   <child link="r_hand_link"/>
+  </joint>
+  <xacro:arm side="l" flip="-1" covers="yes" />
+  <joint name="l_shoulder_out_joint" type="revolute">
+   <axis xyz="1 0 0"/>
+   <limit effort="1000.0" lower="${l_shoulder_out_joint_lower}" upper="${l_shoulder_out_joint_upper}" velocity="${l_shoulder_out_joint_velocity}" />
+   <origin rpy="0 0 0" xyz="0 0.143 0.298"/>
+   <parent link="torso_link"/>
+   <child link="l_shoulder_base_link"/>
+  </joint>
+  <xacro:hand side="l" flip="-1" covers="yes" />
+  <joint name="l_wrist_roll_joint" type="revolute">
+   <axis xyz="0 0 1"/>
+   <limit effort="1000.0" lower="${l_wrist_roll_joint_lower}" upper="${l_wrist_roll_joint_upper}" velocity="${l_wrist_roll_joint_velocity}" />
+   <origin rpy="0 0 0" xyz="-0.0144 -0.01  -0.2885"/>
+   <parent link="l_forearm_link"/>
+   <child link="l_hand_link"/>
+  </joint>
 </robot>
